File: hw/rgb_banner.sch (KiCad schematic (older format))
At the start: 0 parts

Commit message: add 4x ws2812b to schematic
Parts:
- added P1, P2, P3, P4: TST, symbol TST
- added U1, U2, U3, U4: WS2812B, symbol WS2812B
Connections:
- net labels added: +5V, GND, d_in, d_out
- wire segments 0 -> 27
Changed lines of the file:
@@
 LIBS:contrib
 LIBS:valves
+LIBS:kicadlib
+LIBS:rgb_banner-cache
 EELAYER 25 0
 EELAYER END
@@
 Comment4 ""
 $EndDescr
+$Comp
+L WS2812B U1
+U 1 1 556C6577
+P 4050 2100
+F 0 "U1" H 4050 1850 60  0000 C CNN
+F 1 "WS2812B" H 4050 2300 60  0000 C CNN
+F 2 "" H 4350 1950 60  0000 C CNN
+F 3 "" H 4350 1950 60  0000 C CNN
+	1    4050 2100
+	-1   0    0    1
+$EndComp
+$Comp
+L WS2812B U2
+U 1 1 556C661E
+P 5150 2100
+F 0 "U2" H 5150 1850 60  0000 C CNN
+F 1 "WS2812B" H 5150 2300 60  0000 C CNN
+F 2 "" H 5450 1950 60  0000 C CNN
+F 3 "" H 5450 1950 60  0000 C CNN
+	1    5150 2100
+	-1   0    0    1
+$EndComp
+$Comp
+L WS2812B U3
+U 1 1 556C6646
+P 6250 2100
+F 0 "U3" H 6250 1850 60  0000 C CNN
+F 1 "WS2812B" H 6250 2300 60  0000 C CNN
+F 2 "" H 6550 1950 60  0000 C CNN
+F 3 "" H 6550 1950 60  0000 C CNN
+	1    6250 2100
+	-1   0    0    1
+$EndComp
+$Comp
+L WS2812B U4
+U 1 1 556C6673
+P 7350 2100
+F 0 "U4" H 7350 1850 60  0000 C CNN
+F 1 "WS2812B" H 7350 2300 60  0000 C CNN
+F 2 "" H 7650 1950 60  0000 C CNN
+F 3 "" H 7650 1950 60  0000 C CNN
+	1    7350 2100
+	-1   0    0    1
+$EndComp
+Text Label 3350 2500 2    60   ~ 0
++5V
+$Comp
+L GND #PWR01
+U 1 1 556C66A2
+P 3350 1800
+F 0 "#PWR01" H 3350 1800 30  0001 C CNN
+F 1 "GND" H 3350 1730 30  0001 C CNN
+F 2 "" H 3350 1800 60  0000 C CNN
+F 3 "" H 3350 1800 60  0000 C CNN
+	1    3350 1800
+	1    0    0    -1
+$EndComp
+Wire Wire Line
+	3600 2000 3600 1700
+Wire Wire Line
+	3350 1700 5800 1700
+Wire Wire Line
+	3350 1700 3350 1800
+Text Label 3350 2150 2    60   ~ 0
+d_in
+Wire Wire Line
+	3350 2150 3600 2150
+Wire Wire Line
+	3350 2500 7800 2500
+Wire Wire Line
+	4500 2500 4500 2150
+Wire Wire Line
+	4500 2000 4600 2000
+Wire Wire Line
+	4600 2000 4600 2150
+Wire Wire Line
+	4600 2150 4700 2150
+Wire Wire Line
+	5600 2000 5700 2000
+Wire Wire Line
+	5700 2000 5700 2150
+Wire Wire Line
+	5700 2150 5800 2150
+Wire Wire Line
+	5600 2500 5600 2150
+Connection ~ 4500 2500
+Wire Wire Line
+	4700 1700 4700 2000
+Connection ~ 3600 1700
+Wire Wire Line
+	5800 1700 5800 2000
+Connection ~ 4700 1700
+Wire Wire Line
+	5850 1700 6900 1700
+Wire Wire Line
+	6900 1700 6900 2000
+Wire Wire Line
+	6700 2500 6700 2150
+Connection ~ 5600 2500
+Wire Wire Line
+	7800 2500 7800 2150
+Connection ~ 6700 2500
+Wire Wire Line
+	6700 2000 6800 2000
+Wire Wire Line
+	6800 2000 6800 2150
+Wire Wire Line
+	6800 2150 6900 2150
+Text Label 7900 2000 0    60   ~ 0
+d_out
+Wire Wire Line
+	7900 2000 7800 2000
+$Comp
+L TST P1
+U 1 1 556C686B
+P 1850 2100
+F 0 "P1" H 1850 2400 40  0000 C CNN
+F 1 "TST" H 1850 2350 30  0000 C CNN
+F 2 "" H 1850 2100 60  0000 C CNN
+F 3 "" H 1850 2100 60  0000 C CNN
+	1    1850 2100
+	1    0    0    -1
+$EndComp
+$Comp
+L TST P2
+U 1 1 556C69BB
+P 2000 2200
+F 0 "P2" H 2000 2500 40  0000 C CNN
+F 1 "TST" H 2000 2450 30  0000 C CNN
+F 2 "" H 2000 2200 60  0000 C CNN
+F 3 "" H 2000 2200 60  0000 C CNN
+	1    2000 2200
+	1    0    0    -1
+$EndComp
+$Comp
+L TST P3
+U 1 1 556C69DB
+P 2150 2300
+F 0 "P3" H 2150 2600 40  0000 C CNN
+F 1 "TST" H 2150 2550 30  0000 C CNN
+F 2 "" H 2150 2300 60  0000 C CNN
+F 3 "" H 2150 2300 60  0000 C CNN
+	1    2150 2300
+	1    0    0    -1
+$EndComp
+$Comp
+L TST P4
+U 1 1 556C69FA
+P 2300 2400
+F 0 "P4" H 2300 2700 40  0000 C CNN
+F 1 "TST" H 2300 2650 30  0000 C CNN
+F 2 "" H 2300 2400 60  0000 C CNN
+F 3 "" H 2300 2400 60  0000 C CNN
+	1    2300 2400
+	1    0    0    -1
+$EndComp
+Text Label 1850 2200 3    60   ~ 0
++5V
+$Comp
+L GND #PWR02
+U 1 1 556C6A24
+P 2000 2300
+F 0 "#PWR02" H 2000 2300 30  0001 C CNN
+F 1 "GND" H 2000 2230 30  0001 C CNN
+F 2 "" H 2000 2300 60  0000 C CNN
+F 3 "" H 2000 2300 60  0000 C CNN
+	1    2000 2300
+	1    0    0    -1
+$EndComp
+Text Label 2150 2400 3    60   ~ 0
+d_in
+Text Label 2300 2500 3    60   ~ 0
+d_out
+Wire Wire Line
+	2300 2500 2300 2400
+Wire Wire Line
+	2150 2300 2150 2400
+Wire Wire Line
+	2000 2300 2000 2200
+Wire Wire Line
+	1850 2200 1850 2100
 $EndSCHEMATC
