File: hw/rgb_banner.kicad_pcb (KiCad board)
At the start: 2 copper layers, 0 parts

Commit message: schematic pretty much done, start layout
Parts:
- added P1: +5V, kicadlib:TEST_0.100, F.Cu at (276.2, 105.7)
- added P2: GND, kicadlib:TEST_0.100, F.Cu at (276.2, 99.3)
- added P3: DIN, kicadlib:TEST_0.100, F.Cu at (279.6, 105.7)
- added P4: +5V, kicadlib:TEST_0.100, F.Cu at (288.1, 99.3)
- added P5: GND, kicadlib:TEST_0.100, F.Cu at (284.4, 99.3)
- added P6: DOUT, kicadlib:TEST_0.100, F.Cu at (280.3, 99.3)
- added U1: WS2812B, kicadlib:WS2812B_SMD_5050, F.Cu at (72.0, 56.0)
- added U10: WS2812B, kicadlib:WS2812B_SMD_5050, F.Cu at (96.0, 64.0)
- added U11: WS2812B, kicadlib:WS2812B_SMD_5050, F.Cu at (104.0, 64.0)
- added U12: WS2812B, kicadlib:WS2812B_SMD_5050, F.Cu at (112.0, 64.0)
- added U13: WS2812B, kicadlib:WS2812B_SMD_5050, F.Cu at (72.0, 72.0)
- added U14: WS2812B, kicadlib:WS2812B_SMD_5050, F.Cu at (80.0, 72.0)
- added U15: WS2812B, kicadlib:WS2812B_SMD_5050, F.Cu at (88.0, 72.0)
- added U16: WS2812B, kicadlib:WS2812B_SMD_5050, F.Cu at (96.0, 72.0)
- added U17: WS2812B, kicadlib:WS2812B_SMD_5050, F.Cu at (104.0, 72.0)
- added U18: WS2812B, kicadlib:WS2812B_SMD_5050, F.Cu at (112.0, 72.0)
- added U19: WS2812B, kicadlib:WS2812B_SMD_5050, F.Cu at (72.0, 80.0)
- added U2: WS2812B, kicadlib:WS2812B_SMD_5050, F.Cu at (80.0, 56.0)
- added U20: WS2812B, kicadlib:WS2812B_SMD_5050, F.Cu at (80.0, 80.0)
- added U21: WS2812B, kicadlib:WS2812B_SMD_5050, F.Cu at (88.0, 80.0)
- added U22: WS2812B, kicadlib:WS2812B_SMD_5050, F.Cu at (96.0, 80.0)
- added U23: WS2812B, kicadlib:WS2812B_SMD_5050, F.Cu at (104.0, 80.0)
- added U24: WS2812B, kicadlib:WS2812B_SMD_5050, F.Cu at (112.0, 80.0)
- added U25: WS2812B, kicadlib:WS2812B_SMD_5050, F.Cu at (72.0, 88.0)
- added U26: WS2812B, kicadlib:WS2812B_SMD_5050, F.Cu at (80.0, 88.0)
- added U27: WS2812B, kicadlib:WS2812B_SMD_5050, F.Cu at (88.0, 88.0)
- added U28: WS2812B, kicadlib:WS2812B_SMD_5050, F.Cu at (96.0, 88.0)
- added U29: WS2812B, kicadlib:WS2812B_SMD_5050, F.Cu at (104.0, 88.0)
- added U3: WS2812B, kicadlib:WS2812B_SMD_5050, F.Cu at (88.0, 56.0)
- added U30: WS2812B, kicadlib:WS2812B_SMD_5050, F.Cu at (112.0, 88.0)
- added U31: WS2812B, kicadlib:WS2812B_SMD_5050, F.Cu at (72.0, 96.0)
- added U32: WS2812B, kicadlib:WS2812B_SMD_5050, F.Cu at (80.0, 96.0)
- added U33: WS2812B, kicadlib:WS2812B_SMD_5050, F.Cu at (88.0, 96.0)
- added U34: WS2812B, kicadlib:WS2812B_SMD_5050, F.Cu at (96.0, 96.0)
- added U35: WS2812B, kicadlib:WS2812B_SMD_5050, F.Cu at (104.0, 96.0)
- added U36: WS2812B, kicadlib:WS2812B_SMD_5050, F.Cu at (112.0, 96.0)
- added U37: WS2812B, kicadlib:WS2812B_SMD_5050, F.Cu at (72.0, 104.0)
- added U38: WS2812B, kicadlib:WS2812B_SMD_5050, F.Cu at (80.0, 104.0)
- added U39: WS2812B, kicadlib:WS2812B_SMD_5050, F.Cu at (88.0, 104.0)
- added U4: WS2812B, kicadlib:WS2812B_SMD_5050, F.Cu at (96.0, 56.0)
- added U40: WS2812B, kicadlib:WS2812B_SMD_5050, F.Cu at (96.0, 104.0)
- added U41: WS2812B, kicadlib:WS2812B_SMD_5050, F.Cu at (104.0, 104.0)
- added U42: WS2812B, kicadlib:WS2812B_SMD_5050, F.Cu at (112.0, 104.0)
- added U43: WS2812B, kicadlib:WS2812B_SMD_5050, F.Cu at (120.0, 56.0)
- added U44: WS2812B, kicadlib:WS2812B_SMD_5050, F.Cu at (128.0, 56.0)
- added U45: WS2812B, kicadlib:WS2812B_SMD_5050, F.Cu at (136.0, 56.0)
- added U46: WS2812B, kicadlib:WS2812B_SMD_5050, F.Cu at (144.0, 56.0)
- added U47: WS2812B, kicadlib:WS2812B_SMD_5050, F.Cu at (152.0, 56.0)
- added U48: WS2812B, kicadlib:WS2812B_SMD_5050, F.Cu at (160.0, 56.0)
- added U49: WS2812B, kicadlib:WS2812B_SMD_5050, F.Cu at (120.0, 64.0)
- added U5: WS2812B, kicadlib:WS2812B_SMD_5050, F.Cu at (104.0, 56.0)
- added U50: WS2812B, kicadlib:WS2812B_SMD_5050, F.Cu at (128.0, 64.0)
- added U51: WS2812B, kicadlib:WS2812B_SMD_5050, F.Cu at (136.0, 64.0)
- added U52: WS2812B, kicadlib:WS2812B_SMD_5050, F.Cu at (144.0, 64.0)
- added U53: WS2812B, kicadlib:WS2812B_SMD_5050, F.Cu at (152.0, 64.0)
- added U54: WS2812B, kicadlib:WS2812B_SMD_5050, F.Cu at (160.0, 64.0)
- added U55: WS2812B, kicadlib:WS2812B_SMD_5050, F.Cu at (193.7, 63.9)
- added U56: WS2812B, kicadlib:WS2812B_SMD_5050, F.Cu at (202.8, 55.7)
- added U57: WS2812B, kicadlib:WS2812B_SMD_5050, F.Cu at (175.5, 88.5)
- added U58: WS2812B, kicadlib:WS2812B_SMD_5050, F.Cu at (184.6, 80.3)
- added U59: WS2812B, kicadlib:WS2812B_SMD_5050, F.Cu at (193.7, 72.1)
- added U6: WS2812B, kicadlib:WS2812B_SMD_5050, F.Cu at (112.0, 56.0)
- added U60: WS2812B, kicadlib:WS2812B_SMD_5050, F.Cu at (202.8, 63.9)
- added U61: WS2812B, kicadlib:WS2812B_SMD_5050, F.Cu at (211.9, 55.7)
- added U62: WS2812B, kicadlib:WS2812B_SMD_5050, F.Cu at (184.6, 88.5)
- added U63: WS2812B, kicadlib:WS2812B_SMD_5050, F.Cu at (184.0, 40.0)
- added U64: WS2812B, kicadlib:WS2812B_SMD_5050, F.Cu at (211.9, 80.3)
- added U65: WS2812B, kicadlib:WS2812B_SMD_5050, F.Cu at (202.8, 88.5)
- added U66: WS2812B, kicadlib:WS2812B_SMD_5050, F.Cu at (221.0, 63.9)
- added U67: WS2812B, kicadlib:WS2812B_SMD_5050, F.Cu at (211.9, 72.1)
- added U68: WS2812B, kicadlib:WS2812B_SMD_5050, F.Cu at (202.8, 80.3)
- added U69: WS2812B, kicadlib:WS2812B_SMD_5050, F.Cu at (193.7, 88.5)
- added U7: WS2812B, kicadlib:WS2812B_SMD_5050, F.Cu at (72.0, 64.0)
- added U70: WS2812B, kicadlib:WS2812B_SMD_5050, F.Cu at (221.0, 55.7)
- added U71: WS2812B, kicadlib:WS2812B_SMD_5050, F.Cu at (211.9, 63.9)
- added U72: WS2812B, kicadlib:WS2812B_SMD_5050, F.Cu at (221.0, 72.1)
- added U73: WS2812B, kicadlib:WS2812B_SMD_5050, F.Cu at (202.8, 72.1)
- added U74: WS2812B, kicadlib:WS2812B_SMD_5050, F.Cu at (193.7, 80.3)
- added U75: WS2812B, kicadlib:WS2812B_SMD_5050, F.Cu at (230.1, 63.9)
- added U76: WS2812B, kicadlib:WS2812B_SMD_5050, F.Cu at (239.2, 55.7)
- added U77: WS2812B, kicadlib:WS2812B_SMD_5050, F.Cu at (211.9, 88.5)
- added U78: WS2812B, kicadlib:WS2812B_SMD_5050, F.Cu at (221.0, 80.3)
- added U79: WS2812B, kicadlib:WS2812B_SMD_5050, F.Cu at (230.1, 72.1)
- added U8: WS2812B, kicadlib:WS2812B_SMD_5050, F.Cu at (80.0, 64.0)
- added U80: WS2812B, kicadlib:WS2812B_SMD_5050, F.Cu at (239.2, 63.9)
- added U81: WS2812B, kicadlib:WS2812B_SMD_5050, F.Cu at (221.0, 88.5)
- added U82: WS2812B, kicadlib:WS2812B_SMD_5050, F.Cu at (230.1, 80.3)
- added U83: WS2812B, kicadlib:WS2812B_SMD_5050, F.Cu at (230.1, 55.7)
- added U84: WS2812B, kicadlib:WS2812B_SMD_5050, F.Cu at (239.2, 72.1)
- added U9: WS2812B, kicadlib:WS2812B_SMD_5050, F.Cu at (88.0, 64.0)
Other:
- board outline added: 100 x 100 mm

Commit message: work some on pcb, add trial image and link to 200 pcs ws2812b on aliexpress.
Routing:
- net /digit1/+5V: track 0.00 -> 8.01 mm
- added copper zone on F.Cu, net /digit1/+5V
Other:
- outline, holes or cut-outs redrawn
- net class phatty added: clearance 0.254, trace_width 0.45, via_dia 0.889, via_drill 0.635
Changed lines of the file:
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@@
   (general
     (links 255)
-    (no_connects 255)
-    (area 59.949999 49.949999 160.050001 150.050001)
+    (no_connects 252)
+    (area 59.949999 35.841 289.915619 150.050001)
     (thickness 1.6)
-    (drawings 4)
-    (tracks 0)
+    (drawings 7)
+    (tracks 8)
     (zones 0)
     (modules 90)
@@
   (setup
     (last_trace_width 0.254)
+    (user_trace_width 0.45)
     (trace_clearance 0.254)
-    (zone_clearance 0.508)
+    (zone_clearance 0.254)
     (zone_45_only no)
     (trace_min 0.254)
@@
     (uvia_dia 0.508)
     (uvia_drill 0.127)
-    (add_net /digit1/+5V)
     (add_net /digit1/d_in_1)
     (add_net /digit1/d_in_2)
     (add_net /digit1/d_in_3)
     (add_net /digit1/d_in_all)
-    (add_net /digit1/gnd)
     (add_net /digit2/d_in_1)
     (add_net /digit2/d_in_2)
@@
     (add_net "Net-(U83-Pad2)")
   )
+  (net_class phatty ""
+    (clearance 0.254)
+    (trace_width 0.45)
+    (via_dia 0.889)
+    (via_drill 0.635)
+    (uvia_dia 0.508)
+    (uvia_drill 0.127)
+    (add_net /digit1/+5V)
+    (add_net /digit1/gnd)
+  )
   (module kicadlib:TEST_0.100 (layer F.Cu)
     (at 276.152809 105.679)
@@
       (net 78 "Net-(U83-Pad2)"))
   )
+  (gr_line (start 68 52) (end 152.5 52) (angle 90) (layer Edge.Cuts) (width 0.1))
+  (gr_line (start 68 108) (end 125.5 108) (angle 90) (layer Edge.Cuts) (width 0.1))
+  (gr_line (start 68 52) (end 68 108) (angle 90) (layer Edge.Cuts) (width 0.1))
   (gr_line (start 160 50) (end 60 50) (angle 90) (layer Edge.Cuts) (width 0.1))
   (gr_line (start 60 150) (end 60 50) (angle 90) (layer Edge.Cuts) (width 0.1))
   (gr_line (start 160 150) (end 60 150) (angle 90) (layer Edge.Cuts) (width 0.1))
   (gr_line (start 160 50) (end 160 150) (angle 90) (layer Edge.Cuts) (width 0.1))
+  (segment (start 77.55 62.4) (end 77.55 60.95) (width 0.45) (layer F.Cu) (net 5))
+  (segment (start 77.55 60.95) (end 78 60.5) (width 0.45) (layer F.Cu) (net 5))
+  (segment (start 82.45 57.6) (end 82.45 59.45) (width 0.45) (layer F.Cu) (net 5))
+  (segment (start 82.45 59.45) (end 82.5 59.5) (width 0.45) (layer F.Cu) (net 5))
+  (segment (start 74.45 57.6) (end 74.45 59.45) (width 0.45) (layer F.Cu) (net 5))
+  (segment (start 74.45 59.45) (end 74.5 59.5) (width 0.45) (layer F.Cu) (net 5))
+  (segment (start 69.55 62.4) (end 69.55 60.95) (width 0.45) (layer F.Cu) (net 5))
+  (segment (start 69.55 60.95) (end 70 60.5) (width 0.45) (layer F.Cu) (net 5))
+  (zone (net 5) (net_name /digit1/+5V) (layer F.Cu) (hatch edge 0.508)
+    (connect_pads (clearance 0.254))
+    (min_thickness 0.254)
+    (fill yes (arc_segments 16) (thermal_gap 0.254) (thermal_bridge_width 0.255))
+    (polygon
+      (pts
+        (xy 68.5 59) (xy 91 59) (xy 91 61) (xy 68.5 61)
+      )
+    )
+  )
 )

Commit message: pcb layout. zones not working.
Parts:
- moved U76 151.2 mm to (96.0, 104.0), turned to 180 degrees
- moved U75 147.7 mm to (88.0, 104.0), turned to 180 degrees
- moved U61 145.6 mm to (72.0, 96.0)
- moved U73 134.6 mm to (72.0, 104.0), turned to 180 degrees
- moved U80 118.2 mm to (128.0, 104.0), turned to 180 degrees
- moved U64 117.0 mm to (96.0, 96.0)
- moved U74 116.1 mm to (80.0, 104.0), turned to 180 degrees
- moved U79 114.7 mm to (120.0, 104.0), turned to 180 degrees
- moved U66 113.6 mm to (112.0, 96.0)
- moved U78 111.6 mm to (112.0, 104.0), turned to 180 degrees
- moved U63 111.1 mm to (88.0, 96.0)
- moved U77 109.0 mm to (104.0, 104.0), turned to 180 degrees
- moved U62 104.8 mm to (80.0, 96.0)
- moved U65 99.1 mm to (104.0, 96.0)
- moved U67 95.0 mm to (120.0, 96.0)
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Connections:
- net /digit1/d_in_all renamed /d_in
- net /digit2/d_out_all renamed /d_out
- P1 pad 1: /digit1/+5V -> /+5V
- P2 pad 1: /digit1/gnd -> /gnd
- P4 pad 1: /digit1/+5V -> /+5V
- P5 pad 1: /digit1/gnd -> /gnd
- U1 pad 1: /digit1/+5V -> /+5V
- U1 pad 3: /digit1/gnd -> /gnd
- U10 pad 1: /digit1/+5V -> /+5V
- U10 pad 3: /digit1/gnd -> /gnd
- U11 pad 1: /digit1/+5V -> Net-(U11-Pad1)
- U11 pad 2: Net-(U10-Pad4) -> Net-(U11-Pad2)
- U11 pad 3: /digit1/gnd -> /gnd
- U11 pad 4: Net-(U11-Pad4) -> Net-(U10-Pad2)
- U12 pad 1: /digit1/+5V -> /+5V
- U12 pad 2: Net-(U11-Pad4) -> Net-(U12-Pad2)
- U12 pad 3: /digit1/gnd -> /gnd
- U12 pad 4: /digit1/d_in_1 -> Net-(U11-Pad2)
- U13 pad 1: /digit1/+5V -> /+5V
- U13 pad 3: /digit1/gnd -> /gnd
- U14 pad 1: /digit1/+5V -> /+5V
- U14 pad 2: Net-(U14-Pad2) -> Net-(U13-Pad4)
- U14 pad 3: /digit1/gnd -> /gnd
- U14 pad 4: Net-(U13-Pad2) -> Net-(U14-Pad4)
- U15 pad 1: /digit1/+5V -> /+5V
- U15 pad 2: Net-(U15-Pad2) -> Net-(U14-Pad4)
- U15 pad 3: /digit1/gnd -> /gnd
- U15 pad 4: Net-(U14-Pad2) -> Net-(U15-Pad4)
- U16 pad 1: /digit1/+5V -> /+5V
- U16 pad 2: Net-(U16-Pad2) -> Net-(U15-Pad4)
- U16 pad 3: /digit1/gnd -> /gnd
- U16 pad 4: Net-(U15-Pad2) -> Net-(U16-Pad4)
- U17 pad 1: /digit1/+5V -> /+5V
- U17 pad 2: Net-(U17-Pad2) -> Net-(U16-Pad4)
- U17 pad 3: /digit1/gnd -> /gnd
- U17 pad 4: Net-(U16-Pad2) -> Net-(U17-Pad4)
- U18 pad 1: /digit1/+5V -> /+5V
- U18 pad 2: /digit2/d_in_2 -> Net-(U17-Pad4)
- U18 pad 3: /digit1/gnd -> /gnd
- U18 pad 4: Net-(U17-Pad2) -> Net-(U18-Pad4)
- U19 pad 1: /digit1/+5V -> /+5V
- U19 pad 2: Net-(U19-Pad2) -> Net-(U18-Pad4)
- U19 pad 3: /digit1/gnd -> /gnd
- U2 pad 1: /digit1/+5V -> /+5V
- U2 pad 3: /digit1/gnd -> /gnd
- U20 pad 1: /digit1/+5V -> /+5V
- U20 pad 3: /digit1/gnd -> /gnd
- U21 pad 1: /digit1/+5V -> /+5V
- U21 pad 3: /digit1/gnd -> /gnd
- U22 pad 1: /digit1/+5V -> /+5V
- U22 pad 3: /digit1/gnd -> /gnd
- U23 pad 1: /digit1/+5V -> /+5V
- U23 pad 3: /digit1/gnd -> Net-(U23-Pad3)
- U24 pad 1: /digit1/+5V -> /+5V
- U24 pad 3: /digit1/gnd -> /gnd
- U24 pad 4: /digit1/d_in_2 -> Net-(U12-Pad2)
- U25 pad 1: /digit1/+5V -> /+5V
- U25 pad 3: /digit1/gnd -> /gnd
- U25 pad 4: Net-(U19-Pad2) -> Net-(U13-Pad2)
- U26 pad 1: /digit1/+5V -> /+5V
- U26 pad 3: /digit1/gnd -> /gnd
- U27 pad 1: /digit1/+5V -> /+5V
- U27 pad 3: /digit1/gnd -> /gnd
- U28 pad 1: /digit1/+5V -> /+5V
- U28 pad 3: /digit1/gnd -> /gnd
- U29 pad 1: /digit1/+5V -> /+5V
- U29 pad 3: /digit1/gnd -> /gnd
- U3 pad 1: /digit1/+5V -> /+5V
- U3 pad 3: /digit1/gnd -> /gnd
- U30 pad 1: /digit1/+5V -> /+5V
- U30 pad 2: /digit2/d_in_3 -> Net-(U30-Pad2)
- U30 pad 3: /digit1/gnd -> /gnd
- U31 pad 1: /digit1/+5V -> /+5V
- U31 pad 3: /digit1/gnd -> /gnd
- U31 pad 4: Net-(U31-Pad4) -> Net-(U30-Pad2)
- U32 pad 1: /digit1/+5V -> /+5V
- U32 pad 2: Net-(U31-Pad4) -> Net-(U32-Pad2)
- U32 pad 3: /digit1/gnd -> /gnd
- U32 pad 4: Net-(U32-Pad4) -> Net-(U31-Pad2)
- U33 pad 1: /digit1/+5V -> /+5V
- U33 pad 2: Net-(U32-Pad4) -> Net-(U33-Pad2)
- U33 pad 3: /digit1/gnd -> /gnd
- U33 pad 4: Net-(U33-Pad4) -> Net-(U32-Pad2)
- U34 pad 1: /digit1/+5V -> /+5V
- U34 pad 2: Net-(U33-Pad4) -> Net-(U34-Pad2)
- U34 pad 3: /digit1/gnd -> /gnd
- U34 pad 4: Net-(U34-Pad4) -> Net-(U33-Pad2)
- U35 pad 1: /digit1/+5V -> Net-(U35-Pad1)
- U35 pad 2: Net-(U34-Pad4) -> Net-(U35-Pad2)
- U35 pad 3: /digit1/gnd -> /gnd
- U35 pad 4: Net-(U35-Pad4) -> Net-(U34-Pad2)
- U36 pad 1: /digit1/+5V -> /+5V
- U36 pad 2: Net-(U35-Pad4) -> Net-(U36-Pad2)
- U36 pad 3: /digit1/gnd -> /gnd
- U36 pad 4: /digit1/d_in_3 -> Net-(U35-Pad2)
- U37 pad 1: /digit1/+5V -> /+5V
- U37 pad 3: /digit1/gnd -> /gnd
- U37 pad 4: Net-(U31-Pad2) -> Net-(U37-Pad4)
- U38 pad 1: /digit1/+5V -> /+5V
- U38 pad 2: Net-(U38-Pad2) -> Net-(U37-Pad4)
- U38 pad 3: /digit1/gnd -> /gnd
- U38 pad 4: Net-(U37-Pad2) -> Net-(U38-Pad4)
- U39 pad 1: /digit1/+5V -> /+5V
- U39 pad 2: Net-(U39-Pad2) -> Net-(U38-Pad4)
- U39 pad 3: /digit1/gnd -> /gnd
- U39 pad 4: Net-(U38-Pad2) -> Net-(U39-Pad4)
- U4 pad 1: /digit1/+5V -> /+5V
- U4 pad 3: /digit1/gnd -> /gnd
- U40 pad 1: /digit1/+5V -> /+5V
- U40 pad 2: Net-(U40-Pad2) -> Net-(U39-Pad4)
- U40 pad 3: /digit1/gnd -> /gnd
- U40 pad 4: Net-(U39-Pad2) -> Net-(U40-Pad4)
- U41 pad 1: /digit1/+5V -> /+5V
- U41 pad 2: Net-(U41-Pad2) -> Net-(U40-Pad4)
- U41 pad 3: /digit1/gnd -> /gnd
- U41 pad 4: Net-(U40-Pad2) -> Net-(U41-Pad4)
- U42 pad 1: /digit1/+5V -> /+5V
- U42 pad 2: /digit2/d_in_4 -> Net-(U41-Pad4)
- U42 pad 3: /digit1/gnd -> /gnd
- U42 pad 4: Net-(U41-Pad2) -> Net-(U42-Pad4)
- U43 pad 1: /digit1/+5V -> /+5V
- U43 pad 2: Net-(U43-Pad2) -> Net-(U42-Pad4)
- U43 pad 3: /digit1/gnd -> /gnd
- U43 pad 4: /digit2/d_in_1 -> Net-(U43-Pad4)
- U44 pad 1: /digit1/+5V -> /+5V
- U44 pad 2: Net-(U44-Pad2) -> Net-(U43-Pad4)
- U44 pad 3: /digit1/gnd -> /gnd
- U44 pad 4: Net-(U43-Pad2) -> Net-(U44-Pad4)
- U45 pad 1: /digit1/+5V -> /+5V
- U45 pad 2: Net-(U45-Pad2) -> Net-(U44-Pad4)
- U45 pad 3: /digit1/gnd -> /gnd
- U45 pad 4: Net-(U44-Pad2) -> Net-(U45-Pad4)
- U46 pad 1: /digit1/+5V -> /+5V
- U46 pad 2: Net-(U46-Pad2) -> Net-(U45-Pad4)
- U46 pad 3: /digit1/gnd -> /gnd
- U46 pad 4: Net-(U45-Pad2) -> Net-(U46-Pad4)
- U47 pad 1: /digit1/+5V -> /+5V
- U47 pad 2: Net-(U47-Pad2) -> Net-(U46-Pad4)
- U47 pad 3: /digit1/gnd -> Net-(U47-Pad3)
- U47 pad 4: Net-(U46-Pad2) -> Net-(U47-Pad4)
- U48 pad 1: /digit1/+5V -> /+5V
- U48 pad 2: Net-(U48-Pad2) -> Net-(U47-Pad4)
- U48 pad 3: /digit1/gnd -> /gnd
- U48 pad 4: Net-(U47-Pad2) -> Net-(U36-Pad2)
- U49 pad 1: /digit1/+5V -> /+5V
- U49 pad 2: /digit1/d_in_1 -> Net-(U49-Pad2)
- U49 pad 3: /digit1/gnd -> /gnd
- U49 pad 4: Net-(U49-Pad4) -> Net-(U37-Pad2)
- U5 pad 1: /digit1/+5V -> /+5V
- U5 pad 3: /digit1/gnd -> /gnd
- U50 pad 1: /digit1/+5V -> /+5V
- U50 pad 2: Net-(U49-Pad4) -> Net-(U50-Pad2)
- U50 pad 3: /digit1/gnd -> /gnd
- U50 pad 4: Net-(U50-Pad4) -> Net-(U49-Pad2)
- U51 pad 1: /digit1/+5V -> /+5V
- U51 pad 2: Net-(U50-Pad4) -> Net-(U51-Pad2)
- U51 pad 3: /digit1/gnd -> /gnd
- U51 pad 4: Net-(U51-Pad4) -> Net-(U50-Pad2)
- U52 pad 1: /digit1/+5V -> /+5V
- U52 pad 2: Net-(U51-Pad4) -> Net-(U52-Pad2)
- U52 pad 3: /digit1/gnd -> /gnd
- U52 pad 4: Net-(U52-Pad4) -> Net-(U51-Pad2)
- U53 pad 1: /digit1/+5V -> /+5V
- U53 pad 2: Net-(U52-Pad4) -> Net-(U53-Pad2)
- U53 pad 3: /digit1/gnd -> /gnd
- U53 pad 4: Net-(U53-Pad4) -> Net-(U52-Pad2)
- U54 pad 1: /digit1/+5V -> /+5V
- U54 pad 2: Net-(U53-Pad4) -> Net-(U54-Pad2)
- U54 pad 3: /digit1/gnd -> /gnd
- U54 pad 4: Net-(U48-Pad2) -> Net-(U53-Pad2)
- U55 pad 1: /digit1/+5V -> /+5V
- U55 pad 3: /digit1/gnd -> /gnd
- U55 pad 4: /digit2/d_in_2 -> Net-(U54-Pad2)
- U56 pad 1: /digit1/+5V -> /+5V
- U56 pad 3: /digit1/gnd -> /gnd
- U57 pad 1: /digit1/+5V -> /+5V
- U57 pad 3: /digit1/gnd -> /gnd
- U58 pad 1: /digit1/+5V -> /+5V
- U58 pad 3: /digit1/gnd -> /gnd
- U59 pad 1: /digit1/+5V -> Net-(U59-Pad1)
- U59 pad 3: /digit1/gnd -> /gnd
- U6 pad 1: /digit1/+5V -> /+5V
- U6 pad 2: /digit2/d_in_1 -> Net-(U6-Pad2)
- U6 pad 3: /digit1/gnd -> /gnd
- U60 pad 1: /digit1/+5V -> /+5V
- U60 pad 3: /digit1/gnd -> /gnd
- U61 pad 1: /digit1/+5V -> /+5V
- U61 pad 2: /digit1/d_in_2 -> Net-(U61-Pad2)
- U61 pad 3: /digit1/gnd -> /gnd
- U62 pad 1: /digit1/+5V -> /+5V
- U62 pad 3: /digit1/gnd -> /gnd
- U63 pad 1: /digit1/+5V -> /+5V
- U63 pad 3: /digit1/gnd -> /gnd
- U64 pad 1: /digit1/+5V -> /+5V
- U64 pad 3: /digit1/gnd -> /gnd
- U65 pad 1: /digit1/+5V -> /+5V
- U65 pad 3: /digit1/gnd -> /gnd
- U66 pad 1: /digit1/+5V -> /+5V
- U66 pad 3: /digit1/gnd -> /gnd
- U66 pad 4: Net-(U60-Pad2) -> Net-(U66-Pad4)
- U67 pad 1: /digit1/+5V -> /+5V
- U67 pad 2: Net-(U67-Pad2) -> Net-(U66-Pad4)
- U67 pad 3: /digit1/gnd -> /gnd
- U67 pad 4: /digit2/d_in_3 -> Net-(U67-Pad4)
- U68 pad 1: /digit1/+5V -> /+5V
- U68 pad 2: Net-(U68-Pad2) -> Net-(U67-Pad4)
- U68 pad 3: /digit1/gnd -> /gnd
- U68 pad 4: Net-(U67-Pad2) -> Net-(U68-Pad4)
- U69 pad 1: /digit1/+5V -> /+5V
- U69 pad 2: Net-(U69-Pad2) -> Net-(U68-Pad4)
- U69 pad 3: /digit1/gnd -> /gnd
- U69 pad 4: Net-(U68-Pad2) -> Net-(U69-Pad4)
- U7 pad 1: /digit1/+5V -> /+5V
- U7 pad 2: Net-(U13-Pad4) -> Net-(U7-Pad2)
- U7 pad 3: /digit1/gnd -> /gnd
- U7 pad 4: Net-(U7-Pad4) -> Net-(U6-Pad2)
- U70 pad 1: /digit1/+5V -> /+5V
- U70 pad 2: Net-(U70-Pad2) -> Net-(U69-Pad4)
- U70 pad 3: /digit1/gnd -> /gnd
- U70 pad 4: Net-(U69-Pad2) -> Net-(U70-Pad4)
- U71 pad 1: /digit1/+5V -> /+5V
- U71 pad 2: Net-(U71-Pad2) -> Net-(U70-Pad4)
- U71 pad 3: /digit1/gnd -> Net-(U71-Pad3)
- U71 pad 4: Net-(U70-Pad2) -> Net-(U71-Pad4)
- U72 pad 1: /digit1/+5V -> /+5V
- U72 pad 2: Net-(U72-Pad2) -> Net-(U71-Pad4)
- U72 pad 3: /digit1/gnd -> /gnd
- U72 pad 4: Net-(U71-Pad2) -> Net-(U60-Pad2)
- U73 pad 1: /digit1/+5V -> /+5V
- U73 pad 2: /digit1/d_in_3 -> Net-(U73-Pad2)
- U73 pad 3: /digit1/gnd -> /gnd
- U73 pad 4: Net-(U73-Pad4) -> Net-(U61-Pad2)
- U74 pad 1: /digit1/+5V -> /+5V
- U74 pad 2: Net-(U73-Pad4) -> Net-(U74-Pad2)
- U74 pad 3: /digit1/gnd -> /gnd
- U74 pad 4: Net-(U74-Pad4) -> Net-(U73-Pad2)
- U75 pad 1: /digit1/+5V -> /+5V
- U75 pad 2: Net-(U74-Pad4) -> Net-(U75-Pad2)
- U75 pad 3: /digit1/gnd -> /gnd
- U75 pad 4: Net-(U75-Pad4) -> Net-(U74-Pad2)
- U76 pad 1: /digit1/+5V -> /+5V
- U76 pad 2: Net-(U75-Pad4) -> Net-(U76-Pad2)
- U76 pad 3: /digit1/gnd -> /gnd
- U76 pad 4: Net-(U76-Pad4) -> Net-(U75-Pad2)
- U77 pad 1: /digit1/+5V -> /+5V
- U77 pad 2: Net-(U76-Pad4) -> Net-(U77-Pad2)
- U77 pad 3: /digit1/gnd -> /gnd
- U77 pad 4: Net-(U77-Pad4) -> Net-(U76-Pad2)
- U78 pad 1: /digit1/+5V -> /+5V
- U78 pad 2: Net-(U77-Pad4) -> Net-(U78-Pad2)
- U78 pad 3: /digit1/gnd -> /gnd
- U78 pad 4: Net-(U72-Pad2) -> Net-(U77-Pad2)
- U79 pad 1: /digit1/+5V -> /+5V
- U79 pad 3: /digit1/gnd -> /gnd
- U79 pad 4: /digit2/d_in_4 -> Net-(U78-Pad2)
- U8 pad 1: /digit1/+5V -> /+5V
- U8 pad 2: Net-(U7-Pad4) -> Net-(U8-Pad2)
- U8 pad 3: /digit1/gnd -> /gnd
- U8 pad 4: Net-(U8-Pad4) -> Net-(U7-Pad2)
- U80 pad 1: /digit1/+5V -> /+5V
- U80 pad 3: /digit1/gnd -> /gnd
- U81 pad 1: /digit1/+5V -> /+5V
- U81 pad 3: /digit1/gnd -> /gnd
- U82 pad 1: /digit1/+5V -> /+5V
- U82 pad 3: /digit1/gnd -> /gnd
- U83 pad 1: /digit1/+5V -> Net-(U83-Pad1)
- U83 pad 3: /digit1/gnd -> /gnd
- U84 pad 1: /digit1/+5V -> /+5V
- U84 pad 3: /digit1/gnd -> /gnd
- U9 pad 1: /digit1/+5V -> /+5V
- U9 pad 2: Net-(U8-Pad4) -> Net-(U10-Pad4)
- U9 pad 3: /digit1/gnd -> /gnd
- U9 pad 4: Net-(U10-Pad2) -> Net-(U8-Pad2)
Routing:
- net /digit1/+5V: track 8.01 -> 0.00 mm
- net /+5V: track 0.00 -> 8.01 mm
- added copper zone on F.Cu, net /+5V
- added copper zone on F.Cu, net /gnd
Other:
- board size 100 x 100 mm -> 96 x 56 mm

Commit message: add test gerbers
Parts:
- moved P3 94.4 mm to (187.6, 84.7)
- moved P4 94.4 mm to (196.1, 78.3)
- moved P5 94.4 mm to (192.4, 78.3)
- moved P1 94.4 mm to (184.2, 84.7)
- moved P2 94.4 mm to (184.2, 78.3)
- moved P6 94.4 mm to (188.3, 78.3)
Changed lines of the file:
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@@
     (links 248)
     (no_connects 248)
-    (area 67.949999 51.949999 164.050001 108.050001)
+    (area 66.646714 51.841 197.915619 108.050001)
     (thickness 1.6)
     (drawings 4)
@@
     (visible_elements 7FFFF77F)
     (pcbplotparams
-      (layerselection 0x00030_80000001)
+      (layerselection 0x01030_80000001)
       (usegerberextensions false)
       (excludeedgelayer true)
@@
       (outputformat 1)
       (mirror false)
-      (drillshape 1)
+      (drillshape 0)
       (scaleselection 1)
-      (outputdirectory ""))
+      (outputdirectory gerbers))
   )
   (net 0 "")
@@
   )
   (module kicadlib:TEST_0.100 (layer F.Cu)
-    (at 276.152809 105.679)
+    (at 184.152809 84.679)
     (fp_text reference P1 (at 0 -2.1) (layer F.SilkS) hide
       (effects (font (size 1 1) (thickness 0.15)))
@@
   )
   (module kicadlib:TEST_0.100 (layer F.Cu)
-    (at 276.152809 99.279)
+    (at 184.152809 78.279)
     (fp_text reference P2 (at 0 -2.1) (layer F.SilkS) hide
       (effects (font (size 1 1) (thickness 0.15)))
@@
   )
   (module kicadlib:TEST_0.100 (layer F.Cu)
-    (at 279.590904 105.679)
+    (at 187.590904 84.679)
     (fp_text reference P3 (at 0 -2.1) (layer F.SilkS) hide
       (effects (font (size 1 1) (thickness 0.15)))
@@
   )
   (module kicadlib:TEST_0.100 (layer F.Cu)
-    (at 288.062809 99.279)
+    (at 196.062809 78.279)
     (fp_text reference P4 (at 0 -2.1) (layer F.SilkS) hide
       (effects (font (size 1 1) (thickness 0.15)))
@@
   )
   (module kicadlib:TEST_0.100 (layer F.Cu)
-    (at 284.362809 99.279)
+    (at 192.362809 78.279)
     (fp_text reference P5 (at 0 -2.1) (layer F.SilkS) hide
       (effects (font (size 1 1) (thickness 0.15)))
@@
   )
   (module kicadlib:TEST_0.100 (layer F.Cu)
-    (at 280.257571 99.279)
+    (at 188.257571 78.279)
     (fp_text reference P6 (at 0 -2.1) (layer F.SilkS) hide
       (effects (font (size 1 1) (thickness 0.15)))
@@
   (gr_line (start 68 108) (end 164 108) (angle 90) (layer Edge.Cuts) (width 0.1))
   (gr_line (start 68 52) (end 68 108) (angle 90) (layer Edge.Cuts) (width 0.1))
+  (segment (start 77.55 62.4) (end 77.55 60.95) (width 0.45) (layer F.Cu) (net 39))
+  (segment (start 77.55 60.95) (end 78 60.5) (width 0.45) (layer F.Cu) (net 39))
+  (segment (start 82.45 57.6) (end 82.45 59.45) (width 0.45) (layer F.Cu) (net 39))
+  (segment (start 82.45 59.45) (end 82.5 59.5) (width 0.45) (layer F.Cu) (net 39))
+  (segment (start 74.45 57.6) (end 74.45 59.45) (width 0.45) (layer F.Cu) (net 39))
+  (segment (start 74.45 59.45) (end 74.5 59.5) (width 0.45) (layer F.Cu) (net 39))
+  (segment (start 69.55 62.4) (end 69.55 60.95) (width 0.45) (layer F.Cu) (net 39))
   (segment (start 69.55 60.95) (end 70 60.5) (width 0.45) (layer F.Cu) (net 39))
-  (segment (start 69.55 62.4) (end 69.55 60.95) (width 0.45) (layer F.Cu) (net 39))
-  (segment (start 74.45 59.45) (end 74.5 59.5) (width 0.45) (layer F.Cu) (net 39))
-  (segment (start 74.45 57.6) (end 74.45 59.45) (width 0.45) (layer F.Cu) (net 39))
-  (segment (start 82.45 59.45) (end 82.5 59.5) (width 0.45) (layer F.Cu) (net 39))
-  (segment (start 82.45 57.6) (end 82.45 59.45) (width 0.45) (layer F.Cu) (net 39))
-  (segment (start 77.55 60.95) (end 78 60.5) (width 0.45) (layer F.Cu) (net 39))
-  (segment (start 77.55 62.4) (end 77.55 60.95) (width 0.45) (layer F.Cu) (net 39))
   (zone (net 4) (net_name /digit1/+5V) (layer F.Cu) (hatch edge 0.508)
     (connect_pads (clearance 0.254))
@@
     )
   )
+  (zone (net 40) (net_name /gnd) (layer F.Cu) (hatch edge 0.508)
+    (connect_pads (clearance 0.508))
+    (min_thickness 0.254)
+    (fill yes (arc_segments 16) (thermal_gap 0.508) (thermal_bridge_width 0.508))
+    (polygon
+      (pts
+        (xy 163.5 53.5) (xy 68.5 53.5) (xy 68.5 52.5) (xy 163.5 52.5)
+      )
+    )
+  )
+  (zone (net 40) (net_name /gnd) (layer F.Cu) (hatch edge 0.508)
+    (connect_pads (clearance 0.508))
+    (min_thickness 0.254)
+    (fill yes (arc_segments 16) (thermal_gap 0.508) (thermal_bridge_width 0.508))
+    (polygon
+      (pts
+        (xy 163.5 69) (xy 68.5 69) (xy 68.5 67) (xy 163.5 67)
+      )
+    )
+  )
   (zone (net 39) (net_name /+5V) (layer F.Cu) (hatch edge 0.508)
     (connect_pads (clearance 0.508))
@@
     )
   )
+  (zone (net 40) (net_name /gnd) (layer F.Cu) (hatch edge 0.508)
+    (connect_pads (clearance 0.508))
+    (min_thickness 0.254)
+    (fill yes (arc_segments 16) (thermal_gap 0.508) (thermal_bridge_width 0.508))
+    (polygon
+      (pts
+        (xy 163.5 85) (xy 68.5 85) (xy 68.5 83) (xy 163.5 83)
+      )
+    )
+  )
   (zone (net 39) (net_name /+5V) (layer F.Cu) (hatch edge 0.508)
     (connect_pads (clearance 0.508))
@@
     )
   )
-  (zone (net 40) (net_name /gnd) (layer F.Cu) (hatch edge 0.508)
-    (connect_pads (clearance 0.508))
-    (min_thickness 0.254)
-    (fill yes (arc_segments 16) (thermal_gap 0.508) (thermal_bridge_width 0.508))
-    (polygon
-      (pts
-        (xy 163.5 69) (xy 68.5 69) (xy 68.5 67) (xy 163.5 67)
-      )
-    )
-  )
-  (zone (net 40) (net_name /gnd) (layer F.Cu) (hatch edge 0.508)
-    (connect_pads (clearance 0.508))
-    (min_thickness 0.254)
-    (fill yes (arc_segments 16) (thermal_gap 0.508) (thermal_bridge_width 0.508))
-    (polygon
-      (pts
-        (xy 163.5 85) (xy 68.5 85) (xy 68.5 83) (xy 163.5 83)
-      )
-    )
-  )
   (zone (net 39) (net_name /+5V) (layer F.Cu) (hatch edge 0.508)
     (connect_pads (clearance 0.508))
@@
     (polygon
       (pts
-        (xy 163.5 53.5) (xy 68.5 53.5) (xy 68.5 52.5) (xy 163.5 52.5)
+        (xy 163.5 101) (xy 68.5 101) (xy 68.5 99) (xy 163.5 99)
       )
     )
