File: hw/lightBar.kicad_pcb (KiCad board)
At the start: 2 copper layers, 96 x 56 mm, 90 parts, among them P1 +5V, P2 GND, P3 DIN, P4 +5V, P5 GND, P6 DOUT, U1 WS2812B, U10 WS2812B, U11 WS2812B, U12 WS2812B, U13 WS2812B, U14 WS2812B, U15 WS2812B, U16 WS2812B, U17 WS2812B, U18 WS2812B, U19 WS2812B, U2 WS2812B, U20 WS2812B, U21 WS2812B, U22 WS2812B, U23 WS2812B, U24 WS2812B, U25 WS2812B, U26 WS2812B, U27 WS2812B, U28 WS2812B, U29 WS2812B, U3 WS2812B, U30 WS2812B, U31 WS2812B, U32 WS2812B, U33 WS2812B, U34 WS2812B, U35 WS2812B, U36 WS2812B, U37 WS2812B, U38 WS2812B, U39 WS2812B, U4 WS2812B, U40 WS2812B, U41 WS2812B, U42 WS2812B, U43 WS2812B, U44 WS2812B, U45 WS2812B, U46 WS2812B, U47 WS2812B, U48 WS2812B, U49 WS2812B, U5 WS2812B, U50 WS2812B, U51 WS2812B, U52 WS2812B, U53 WS2812B, U54 WS2812B, U55 WS2812B, U56 WS2812B, U57 WS2812B, U58 WS2812B, U59 WS2812B, U6 WS2812B, U60 WS2812B, U61 WS2812B, U62 WS2812B, U63 WS2812B, U64 WS2812B, U65 WS2812B, U66 WS2812B, U67 WS2812B, U68 WS2812B, U69 WS2812B, U7 WS2812B, U70 WS2812B, U71 WS2812B, U72 WS2812B, U73 WS2812B, U74 WS2812B, U75 WS2812B, U76 WS2812B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

Commit message: renames
Other:
- board text added: "RGB Banner 2 Digit Module https://github.com/noahp/lightBar PCB Rev 0.1"
- board text removed: "RGB Banner 2 Digit Module https://github.com/noahp/rgb_banner PCB Rev 0.1"
Changed lines of the file:
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@@
       (net 37 "Net-(U83-Pad2)"))
   )
-  (gr_text "RGB Banner 2 Digit Module\nhttps://github.com/noahp/rgb_banner\nPCB Rev 0.1" (at 112 61.5) (layer B.SilkS)
+  (gr_text "RGB Banner 2 Digit Module\nhttps://github.com/noahp/lightBar\nPCB Rev 0.1" (at 112 61.5) (layer B.SilkS)
     (effects (font (size 2 2) (thickness 0.35)) (justify mirror))
   )

Commit message: replot
Other:
- board text added: "LightBar 2 Digit Module https://github.com/noahp/lightBar PCB Rev 0.1"
- board text removed: "RGB Banner 2 Digit Module https://github.com/noahp/lightBar PCB Rev 0.1"

Commit message: fix some errors in the pcb- unconnected pads >_< change version silk to 2
Routing:
- net /+5V: track 433.9 -> 442.8 mm
Other:
- board text added: "LightBar 2 Digit Module https://github.com/noahp/lightBar PCB Rev 2"
- board text removed: "LightBar 2 Digit Module https://github.com/noahp/lightBar PCB Rev 0.1"
